Commit message: working setup for franka (modified srdf and launch file for correct franka hand attachment) also edited the ros2_control for fake robot hardware (effort -> joint position) since initially there where no joint position update with effort in fake hardware

File: franka_moveit_config/srdf/panda_arm.srdf.xacro (robot description, xacro)
@@ -5,5 +5,5 @@
   <xacro:property name="arm_id" value="$(arg arm_id)"/>
   <xacro:include filename="$(find franka_moveit_config)/srdf/panda_arm.xacro"/>
-  <xacro:panda_arm arm_id="${arm_id}"/>
+  <xacro:panda_arm arm_id="${arm_id}" hand="$(arg hand)"/>
   <xacro:if value="$(arg hand)">
     <xacro:include filename="$(find franka_moveit_config)/srdf/hand.xacro"/>

File: franka_moveit_config/srdf/panda_arm.xacro (robot description, xacro)
@@ -1,7 +1,12 @@
 <?xml version="1.0" ?>
 <robot xmlns:xacro="http://www.ros.org/wiki/xacro" name="panda">
-  <xacro:macro name="panda_arm" params="arm_id:='panda' ">
+  <xacro:macro name="panda_arm" params="arm_id:='panda' hand:='true'">
     <xacro:include filename="$(find franka_moveit_config)/srdf/group_definition.xacro"/>
-    <xacro:group_definition arm_id="${arm_id}" group_name="${arm_id}_manipulator" tip_link="${arm_id}_hand_tcp"/>
+    <xacro:if value="${hand}">
+      <xacro:group_definition arm_id="${arm_id}" group_name="${arm_id}_manipulator" tip_link="${arm_id}_hand_tcp"/>
+    </xacro:if>
+    <xacro:unless value="${hand}">
+      <xacro:group_definition arm_id="${arm_id}" group_name="${arm_id}_manipulator" tip_link="${arm_id}_link8"/>
+    </xacro:unless>
     <xacro:group_definition arm_id="${arm_id}" group_name="${arm_id}_arm" tip_link="${arm_id}_link8"/>
     <virtual_joint name="virtual_joint" type="fixed" parent_frame="world" child_link="${arm_id}_link0"/>
