Commit message: thinkgrasp working setup!

File: franka_moveit_config/srdf/panda_arm.xacro (robot description, xacro)
@@ -10,4 +10,13 @@
     </xacro:unless>
     <xacro:group_definition arm_id="${arm_id}" group_name="${arm_id}_arm" tip_link="${arm_id}_link8"/>
+    <group_state name="home" group="${arm_id}_arm">
+      <joint name="${arm_id}_joint1" value="0.0"/>
+      <joint name="${arm_id}_joint2" value="-0.78539816"/>
+      <joint name="${arm_id}_joint3" value="0.0"/>
+      <joint name="${arm_id}_joint4" value="-2.35619449"/>
+      <joint name="${arm_id}_joint5" value="0.0"/>
+      <joint name="${arm_id}_joint6" value="1.57079633"/>
+      <joint name="${arm_id}_joint7" value="0.78539816"/>
+    </group_state>
     <virtual_joint name="virtual_joint" type="fixed" parent_frame="world" child_link="${arm_id}_link0"/>
     <disable_collisions link1="${arm_id}_link0" link2="${arm_id}_link1" reason="Adjacent"/>
