Commit message: control interfaces for isaac sim franka hardware

File: franka_description/robots/panda_arm.ros2_control.xacro (robot description, xacro)
@@ -1,15 +1,22 @@
 <?xml version="1.0"?>
 <robot xmlns:xacro="http://www.ros.org/wiki/xacro">
-  <xacro:macro name="panda_arm_ros2_control" params="ns robot_ip use_fake_hardware:=^|false fake_sensor_commands:=^|false">
+  <xacro:macro name="panda_arm_ros2_control" params="ns robot_ip use_fake_hardware:=^|false fake_sensor_commands:=^|false use_isaac_sim:=^|false">
     <ros2_control name="FrankaHardwareInterface" type="system">
       <hardware>
-        <xacro:if value="${use_fake_hardware}">
-          <plugin>fake_components/GenericSystem</plugin>
-          <param name="fake_sensor_commands">${fake_sensor_commands}</param>
-          <param name="state_following_offset">0.0</param>
+        <xacro:if value="${use_isaac_sim}">
+          <plugin>topic_based_ros2_control/TopicBasedSystem</plugin>
+          <param name="joint_commands_topic">/panda_joint_commands</param>
+          <param name="joint_states_topic">/joint_states</param>
         </xacro:if>
-        <xacro:unless value="${use_fake_hardware}">
-          <plugin>franka_hardware/FrankaHardwareInterface</plugin>
-          <param name="robot_ip">${robot_ip}</param>
+        <xacro:unless value="${use_isaac_sim}">
+          <xacro:if value="${use_fake_hardware}">
+            <plugin>fake_components/GenericSystem</plugin>
+            <param name="fake_sensor_commands">${fake_sensor_commands}</param>
+            <param name="state_following_offset">0.0</param>
+          </xacro:if>
+          <xacro:unless value="${use_fake_hardware}">
+            <plugin>franka_hardware/FrankaHardwareInterface</plugin>
+            <param name="robot_ip">${robot_ip}</param>
+          </xacro:unless>
         </xacro:unless>
       </hardware>

File: franka_description/robots/panda_arm.urdf.xacro (robot description, xacro)
@@ -6,4 +6,5 @@
   <xacro:arg name="use_fake_hardware" default="false"/>
   <xacro:arg name="fake_sensor_commands" default="false"/>
+  <xacro:arg name="use_isaac_sim" default="false"/>
   <xacro:include filename="$(find franka_description)/robots/panda_arm.xacro"/>
   <xacro:panda_arm arm_id="$(arg arm_id)" safety_distance="0.03"/>
@@ -13,4 +14,4 @@
   </xacro:if>
   <xacro:include filename="$(find franka_description)/robots/panda_arm.ros2_control.xacro"/>
-  <xacro:panda_arm_ros2_control ns="$(arg arm_id)" robot_ip="$(arg robot_ip)" use_fake_hardware="$(arg use_fake_hardware)" fake_sensor_commands="$(arg fake_sensor_commands)"/>
+  <xacro:panda_arm_ros2_control ns="$(arg arm_id)" robot_ip="$(arg robot_ip)" use_fake_hardware="$(arg use_fake_hardware)" fake_sensor_commands="$(arg fake_sensor_commands)" use_isaac_sim="$(arg use_isaac_sim)"/>
 </robot>

Commit message: edit gripper files

File: franka_description/robots/panda_arm.ros2_control.xacro (robot description, xacro)
@@ -1,5 +1,5 @@
 <?xml version="1.0"?>
 <robot xmlns:xacro="http://www.ros.org/wiki/xacro">
-  <xacro:macro name="panda_arm_ros2_control" params="ns robot_ip use_fake_hardware:=^|false fake_sensor_commands:=^|false use_isaac_sim:=^|false">
+  <xacro:macro name="panda_arm_ros2_control" params="ns robot_ip use_fake_hardware:=^|false fake_sensor_commands:=^|false use_isaac_sim:=^|false load_gripper:=^|false">
     <ros2_control name="FrankaHardwareInterface" type="system">
       <hardware>
@@ -46,4 +46,17 @@
       <xacro:configure_joint joint_name="${ns}_joint6" initial_position="${pi/2}"/>
       <xacro:configure_joint joint_name="${ns}_joint7" initial_position="${pi/4}"/>
+      <xacro:if value="${use_isaac_sim and load_gripper}">
+        <joint name="${ns}_finger_joint1">
+          <param name="initial_position">0.035</param>
+          <command_interface name="position"/>
+          <state_interface name="position"/>
+          <state_interface name="velocity"/>
+        </joint>
+        <joint name="${ns}_finger_joint2">
+          <param name="initial_position">0.035</param>
+          <state_interface name="position"/>
+          <state_interface name="velocity"/>
+        </joint>
+      </xacro:if>
     </ros2_control>
   </xacro:macro>

File: franka_description/robots/panda_arm.urdf.xacro (robot description, xacro)
@@ -14,4 +14,4 @@
   </xacro:if>
   <xacro:include filename="$(find franka_description)/robots/panda_arm.ros2_control.xacro"/>
-  <xacro:panda_arm_ros2_control ns="$(arg arm_id)" robot_ip="$(arg robot_ip)" use_fake_hardware="$(arg use_fake_hardware)" fake_sensor_commands="$(arg fake_sensor_commands)" use_isaac_sim="$(arg use_isaac_sim)"/>
+  <xacro:panda_arm_ros2_control ns="$(arg arm_id)" robot_ip="$(arg robot_ip)" use_fake_hardware="$(arg use_fake_hardware)" fake_sensor_commands="$(arg fake_sensor_commands)" use_isaac_sim="$(arg use_isaac_sim)" load_gripper="$(arg hand)"/>
 </robot>
